Commit message: model is now can imported to the isaacsim but rotors are all at same origin point.

File: extensions/pegasus.simulator/pegasus/simulator/assets/Robots/x500/model.urdf (robot description, URDF)
Before this commit: robot x500, 5 links, 4 joints
Links:
- link base_link: mass None -> 2.0; geometry collision box size=0.015 0.015 0.21; collision box size=0.015 0.015 0.21
- link rotor0: mass None -> 0.016076923076923075; geometry collision box size=0.2792307692307692 0.016923076923076923 0.00084615384615384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; visual mesh filename=meshes/1345_prop_ccw.stl scale=0.8461538461538461 0.8461538461538461 0.8461538461538461
- link rotor1: mass None -> 0.016076923076923075; geometry collision box size=0.2792307692307692 0.016923076923076923 0.00084615384615384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; visual mesh filename=meshes/1345_prop_ccw.stl scale=0.8461538461538461 0.8461538461538461 0.8461538461538461
- link rotor2: mass None -> 0.016076923076923075; geometry collision box size=0.2792307692307692 0.016923076923076923 0.00084615384615384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; visual mesh filename=meshes/1345_prop_cw.stl scale=0.8461538461538461 0.8461538461538461 0.8461538461538461
- link rotor3: mass None -> 0.016076923076923075; geometry collision box size=0.2792307692307692 0.016923076923076923 0.00084615384615384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; visual mesh filename=meshes/1345_prop_cw.stl scale=0.8461538461538461 0.8461538461538461 0.8461538461538461
Joints:
- joint joint0: child  -> rotor0; parent  -> base_link
- joint joint1: child  -> rotor1; parent  -> base_link
- joint joint2: child  -> rotor2; parent  -> base_link
- joint joint3: child  -> rotor3; parent  -> base_link

Commit message: model is now successfully imprted to isaacsim

File: extensions/pegasus.simulator/pegasus/simulator/assets/Robots/x500/model.urdf (robot description, URDF)
Before this commit: robot x500, 5 links, 4 joints
Joints:
- joint joint0: origin (none) -> xyz=0.174 -0.174 0.06 rpy=0 0 0
- joint joint1: origin (none) -> xyz=-0.174 0.174 0.06 rpy=0 0 0
- joint joint2: origin (none) -> xyz=0.174 0.174 0.06 rpy=0 0 0
- joint joint3: origin (none) -> xyz=-0.174 -0.174 0.06 rpy=0 0 0

Commit message: model urdf is finally fixed. also the axis is set to x but need to be z. can change it in the isaacsim gui. s500_generic is also done

File: extensions/pegasus.simulator/pegasus/simulator/assets/Robots/x500/model.urdf (robot description, URDF)
Before this commit: robot x500, 5 links, 4 joints
Links:
- removed link base_link
- added link body, mass 2.0; collision box size=0.015 0.015 0.21; collision box size=0.015 0.015 0.21
Joints:
- joint joint0: parent base_link -> body
- joint joint1: parent base_link -> body
- joint joint2: parent base_link -> body
- joint joint3: parent base_link -> body
